Commit message: Merging with https://github.com/PepperlFuchs/pf_lidar_ros_driver.git

File: pf_description/urdf/r2000.urdf.xacro (robot description, xacro)
@@ -2,5 +2,5 @@
 <robot xmlns:xacro="http://ros.org/wiki/xacro">
     <xacro:macro name="r2000" params="prefix" >
-        <link name="${prefix}base_link" >
+        <link name="${prefix}scanner_link" >
             <visual>
                 <origin xyz="0 0 0" rpy="1.57 0 1.57" />

File: pf_description/urdf/r2000_world.urdf.xacro (robot description, xacro)
@@ -6,8 +6,8 @@
     <!-- instantiate r2300 macro -->
     <xacro:r2000 prefix="" />
-    <!-- connect world link to scanner base_link -->
+    <!-- connect world link to scanner link -->
     <joint name="world_joint" type="fixed">
         <parent link="world" />
-        <child link = "base_link" />
+        <child link = "scanner_link" />
         <origin xyz="0.0 0.0 0.0" rpy="0.0 0.0 0.0" />
     </joint>

File: pf_description/urdf/r2300.urdf.xacro (robot description, xacro)
@@ -2,5 +2,5 @@
 <robot xmlns:xacro="http://ros.org/wiki/xacro">
     <xacro:macro name="r2300" params="prefix" >
-        <link name="${prefix}base_link" >
+        <link name="${prefix}scanner_link" >
             <visual>
                 <origin xyz="-0.00195 0.0158 -0.0094" rpy="-1.57 0 1.57" />

File: pf_description/urdf/r2300_world.urdf.xacro (robot description, xacro)
@@ -6,8 +6,8 @@
     <!-- instantiate r2300 macro -->
     <xacro:r2300 prefix="" />
-    <!-- connect world link to scanner base_link -->
+    <!-- connect world link to scanner link -->
     <joint name="world_joint" type="fixed">
         <parent link="world" />
-        <child link = "base_link" />
+        <child link = "scanner_link" />
         <origin xyz="0.0 0.0 0.0" rpy="0.0 0.0 0.0" />
     </joint>
